Commit message: update

File: aerial_motion/squeeze_navigation/urdf/ceiling_opening.urdf (robot description, URDF)
Before this commit: robot opening, 0 links, 2 joints
Joints:
- removed joint frame_joint2
- added joint frame_joint4: type fixed, parent main_frame1, child main_frame5, origin xyz=0 0 0 rpy=0 0 0, axis 0 0 1
- added joint frame_joint5: type fixed, parent main_frame1, child main_frame6, origin xyz=0 0 0 rpy=0 0 0, axis 0 0 1
- added joint frame_joint6: type fixed, parent main_frame1, child main_frame7, origin xyz=0 0 0 rpy=0 0 0, axis 0 0 1

Commit message: update

File: aerial_motion/squeeze_navigation/urdf/ceiling_opening.urdf (robot description, URDF)
Before this commit: robot opening, 0 links, 4 joints
Joints:
- removed joint frame_joint6
